Commit message: bug fixed

File: delto_3f_description/urdf/delto_3f.urdf.xacro (robot description, xacro)
@@ -1,5 +1,5 @@
 <?xml version="1.0" ?>
 <robot xmlns:xacro="http://www.ros.org/wiki/xacro">
-    <xacro:macro name="insert_gripper" params="prefix parent *origin">
+    <xacro:macro name="insert_gripper" params="prefix:='' parent *origin">
         <material name="silver">
             <color rgba="0.700 0.700 0.700 1.000"/>
